File: cb-ld/cb-ld.sch (KiCad schematic (older format))
At the start: 35 parts, among them P1 CONN_01X14, P2 CONN_01X14, U1 MBC13917, U4 CC1190

Commit message: External LNA removed from design
Parts:
- removed C1, C2: 47p, mysmd:SM0603S, symbol C
- removed C21: 3p, mysmd:SM0603S, symbol C
- removed C3: 2p, mysmd:SM0603S, symbol C
- removed C4: 100n, mysmd:SM0603S, symbol C
- removed L6: 6.8n, mysmd:SM0603S, symbol INDUCTOR
- removed L7: 10n, mysmd:SM0603S, symbol INDUCTOR
- removed U1: MBC13917, mysmd:MLPD-6, symbol MBC13917
- C10, C11, C12, C13, C14, C15, C16, C17, C18, C19, C20, C5, C6, C7, C8, C9: symbol C -> C-RESCUE-cb-ld
- R1: symbol R -> R-RESCUE-cb-ld
Connections:
- net LNA_A: no longer names the net of C13.1, C19.1, L4.2, L5.2
- net LNA_B: no longer names the net of C11.1, C15.2, U4.4 (TR_SW)
- net LNA_C: no longer names the net of C11.2, U4.5 (LNA_IN)
Other:
- note removed: "Not populated"
