File: rpishield/rpishield.sch (KiCad schematic (older format))
At the start: 15 parts, among them P1 CONN_13X2, P2 CONN_01X09, U1 ANTENNA, U2 DS1338, U3 MCP1702, X1 32.768KHz

Commit message: RPi shield for panStamp 2 completed
Parts:
- C1: value 4.7u -> 10u
Changed lines of the file:
@@
 EESchema Schematic File Version 2
-LIBS:rpishield-rescue
 LIBS:power
 LIBS:device
@@
 LIBS:memory
 LIBS:xilinx
+LIBS:special
 LIBS:microcontrollers
 LIBS:dsp
@@
 P 2550 6200
 F 0 "C1" H 2600 6300 50  0000 L CNN
-F 1 "4.7u" H 2600 6100 50  0000 L CNN
+F 1 "10u" H 2600 6100 50  0000 L CNN
 F 2 "mysmd:SM0603S" H 2550 6200 60  0001 C CNN
 F 3 "" H 2550 6200 60  0001 C CNN
