File: esp-matrix/esp-matrix.sch (KiCad schematic (older format))
At the start: 14 parts, among them SW1 SW_PUSH_SMALL, SW2 SW_PUSH_SMALL, U1 ESP-12E, U2 MCP1702-3.3

Commit message: First version finished
Parts:
- added D1: D_Schottky_x2_ACom_KKA, mysmd:SOT23, symbol D_Schottky_x2_ACom_KKA
- added F1: FUSE, libcms:SM0805, symbol FUSE
- added P1: CONN_02X08, Pin_Headers:Pin_Header_Straight_2x08, symbol CONN_02X08
- added P2: CONN_01X02, myconnectors:terminal_block_5mm_2P, symbol CONN_01X02
- added U10, U11, U4, U5, U6, U7, U8, U9: 74AHC1G34, libcms:SOT23-5, symbol 74AHC1G34
- U3: renamed from U?; footprint Housings_SOT-23_SOT-143_TSOT-6:SOT-23-5 -> libcms:SOT23-5
Connections:
- net +5V: now also D1.1 (K), D1.2 (K), F1.2, U10.5 (VCC), U11.5 (VCC), U4.5 (VCC), U5.5 (VCC), U6.5 (VCC), U7.5 (VCC), U8.5 (VCC), U9.5 (VCC)
- net GND: now also D1.3 (A), P1.1 (P1), P1.13 (P13), P1.15 (P15), P1.3 (P3), P1.5 (P5), P2.1 (P1), U10.3 (GND), U11.3 (GND), U4.3 (GND), U5.3 (GND), U6.3 (GND), U7.3 (GND), U8.3 (GND), U9.3 (GND)
- net GPIO0: now also U4.2
- net GPIO12: now also U10.2
- net GPIO13: now also U8.2
- net GPIO14: now also U7.2
- net GPIO15: now also U3.2
- net GPIO16: now also U6.2; no longer U3.2
- net GPIO2: now also U5.2
- net GPIO4: now also U11.2
- net GPIO5: now also U9.2
- net EN: now reaches U3.4
- net EN: now also P1.7 (P7)
- new net: F1.1, P2.2 (P2)
- new net LA: P1.2 (P2), U6.4
- new net LB: P1.4 (P4), U7.4
- new net LC: P1.6 (P6), U10.4
- new net LD: P1.8 (P8), U8.4
- new net LT: P1.14 (P14), U11.4
- new net R1: P1.9 (P9), U4.4
- new net R2: P1.11 (P11), U5.4
- new net SK: P1.16 (P16), U9.4
- no-connect marks 6 -> 8
Other:
- moved on the sheet: C1, C2, C3, C4, C5, PROG1, R2, R4, R8, SW1, SW2, U1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
