File: cb-rgb/cb-rgb.sch (KiCad schematic (older format))
At the start: 14 parts, among them P1 CONN_01X14, P2 CONN_01X14, P3 CONN_8, Q1 MOS_N, Q2 MOS_N, Q3 MOS_N, U2 UA78M33

Commit message: PWM pins fixed
Parts:
- added SW1: SW_PUSH, mysmd:switch-tact-noah, symbol SW_PUSH
Connections:
- net D4 is gone; now on net BLUE_CH: P2.7 (P7), PS1.18 (D4/P1.4/I2C_SCL/PWM)
- net BLUE_CH: no longer P2.2 (P2), PS1.23 (D22/P3.6)
- net D19: now also Q1.G
- net D20: no longer Q1.G
- net D21: no longer Q2.G
- net D3: now also Q2.G
- net GND: now also SW1.1
- net RESET: now also SW1.2
- new net D22: P2.2 (P2), PS1.23 (D22/P3.6)
Changed lines of the file:
@@
 	1    0    0    -1
 $EndComp
-Text Label 4950 3100 2    60   ~ 0
+Text Label 1250 2900 0    60   ~ 0
 GREEN_CH
 Text Label 7600 3150 0    60   ~ 0
@@
 	1    0    0    -1
 $EndComp
-Text Label 4950 3200 2    60   ~ 0
+Text Label 1250 2800 0    60   ~ 0
 BLUE_CH
-Text Label 4950 3000 2    60   ~ 0
+Text Label 4950 2900 2    60   ~ 0
 RED_CH
 $Comp
-L GND-RESCUE-cb-rgb #PWR03
+L GND-RESCUE-cb-rgb #PWR02
 U 1 1 48C4C07A
 P 7250 3500
-F 0 "#PWR03" H 7250 3500 30  0001 C CNN
+F 0 "#PWR02" H 7250 3500 30  0001 C CNN
 F 1 "GND" H 7250 3430 30  0001 C CNN
 F 2 "" H 7250 3500 60  0001 C CNN
@@
 $EndComp
 $Comp
-L GND-RESCUE-cb-rgb #PWR04
+L GND-RESCUE-cb-rgb #PWR03
 U 1 1 48C4C075
 P 8400 3500
-F 0 "#PWR04" H 8400 3500 30  0001 C CNN
+F 0 "#PWR03" H 8400 3500 30  0001 C CNN
 F 1 "GND" H 8400 3430 30  0001 C CNN
 F 2 "" H 8400 3500 60  0001 C CNN
@@
 $EndComp
 $Comp
-L GND-RESCUE-cb-rgb #PWR05
+L GND-RESCUE-cb-rgb #PWR04
 U 1 1 48C4C06D
 P 9550 3500
-F 0 "#PWR05" H 9550 3500 30  0001 C CNN
+F 0 "#PWR04" H 9550 3500 30  0001 C CNN
 F 1 "GND" H 9550 3430 30  0001 C CNN
 F 2 "" H 9550 3500 60  0001 C CNN
@@
 $EndComp
 $Comp
-L GND-RESCUE-cb-rgb #PWR06
+L GND-RESCUE-cb-rgb #PWR05
 U 1 1 48B3CC0B
 P 4850 7000
-F 0 "#PWR06" H 4850 7000 30  0001 C CNN
+F 0 "#PWR05" H 4850 7000 30  0001 C CNN
 F 1 "GND" H 4850 6930 30  0001 C CNN
 F 2 "" H 4850 7000 60  0001 C CNN
@@
 $EndComp
 $Comp
-L GND-RESCUE-cb-rgb #PWR07
+L GND-RESCUE-cb-rgb #PWR06
 U 1 1 48B2DC35
 P 3200 7000
-F 0 "#PWR07" H 3200 7000 30  0001 C CNN
+F 0 "#PWR06" H 3200 7000 30  0001 C CNN
 F 1 "GND" H 3200 6930 30  0001 C CNN
 F 2 "" H 3200 7000 60  0001 C CNN
@@
 $EndComp
 $Comp
-L GND-RESCUE-cb-rgb #PWR08
+L GND-RESCUE-cb-rgb #PWR07
 U 1 1 48B2D42A
 P 2550 7000
-F 0 "#PWR08" H 2550 7000 30  0001 C CNN
+F 0 "#PWR07" H 2550 7000 30  0001 C CNN
 F 1 "GND" H 2550 6930 30  0001 C CNN
 F 2 "" H 2550 7000 60  0001 C CNN
@@
 $EndComp
 $Comp
-L GND-RESCUE-cb-rgb #PWR09
+L GND-RESCUE-cb-rgb #PWR08
 U 1 1 48B2D427
 P 3900 7000
-F 0 "#PWR09" H 3900 7000 30  0001 C CNN
+F 0 "#PWR08" H 3900 7000 30  0001 C CNN
 F 1 "GND" H 3900 6930 30  0001 C CNN
 F 2 "" H 3900 7000 60  0001 C CNN
@@
 $EndComp
 $Comp
-L GND-RESCUE-cb-rgb #PWR010
+L GND-RESCUE-cb-rgb #PWR09
 U 1 1 48B2D41E
 P 4400 7000
-F 0 "#PWR010" H 4400 7000 30  0001 C CNN
+F 0 "#PWR09" H 4400 7000 30  0001 C CNN
 F 1 "GND" H 4400 6930 30  0001 C CNN
 F 2 "" H 4400 7000 60  0001 C CNN
@@
 RESET
 $Comp
-L VCC #PWR011
+L VCC #PWR010
 U 1 1 55D4AFFB
 P 8600 5550
-F 0 "#PWR011" H 8600 5650 30  0001 C CNN
+F 0 "#PWR010" H 8600 5650 30  0001 C CNN
 F 1 "VCC" H 8600 5650 30  0000 C CNN
 F 2 "" H 8600 5550 60  0001 C CNN
@@
 D6
 $Comp
-L GND #PWR012
+L GND #PWR011
 U 1 1 55D4B00B
 P 7300 5650
-F 0 "#PWR012" H 7300 5650 30  0001 C CNN
+F 0 "#PWR011" H 7300 5650 30  0001 C CNN
 F 1 "GND" H 7300 5580 30  0001 C CNN
 F 2 "" H 7300 5650 60  0001 C CNN
@@
 D4
 $Comp
-L GND #PWR013
+L GND #PWR012
 U 1 1 55D4B014
 P 8300 5450
-F 0 "#PWR013" H 8300 5450 30  0001 C CNN
+F 0 "#PWR012" H 8300 5450 30  0001 C CNN
 F 1 "GND" H 8300 5380 30  0001 C CNN
 F 2 "" H 8300 5450 60  0001 C CNN
@@
 $EndComp
 $Comp
-L GND #PWR014
+L GND #PWR013
 U 1 1 55D4B1D1
 P 5700 4550
-F 0 "#PWR014" H 5700 4550 30  0001 C CNN
+F 0 "#PWR013" H 5700 4550 30  0001 C CNN
 F 1 "GND" H 5700 4480 30  0001 C CNN
 F 2 "" H 5700 4550 60  0001 C CNN
@@
 $EndComp
 $Comp
-L GND #PWR015
+L GND #PWR014
 U 1 1 55D4B1F6
 P 5700 5250
-F 0 "#PWR015" H 5700 5250 30  0001 C CNN
+F 0 "#PWR014" H 5700 5250 30  0001 C CNN
 F 1 "GND" H 5700 5180 30  0001 C CNN
 F 2 "" H 5700 5250 60  0001 C CNN
@@
 	5700 5250 5650 5250
 $Comp
-L +12V #PWR016
+L +12V #PWR015
 U 1 1 55D4B5F1
 P 5950 4600
-F 0 "#PWR016" H 5950 4550 20  0001 C CNN
+F 0 "#PWR015" H 5950 4550 20  0001 C CNN
 F 1 "+12V" H 5950 4700 30  0000 C CNN
 F 2 "" H 5950 4600 60  0001 C CNN
@@
 	5650 5050 6200 5050
 $Comp
-L GND #PWR017
+L GND #PWR016
 U 1 1 55D4BD9E
 P 5700 5150
-F 0 "#PWR017" H 5700 5150 30  0001 C CNN
+F 0 "#PWR016" H 5700 5150 30  0001 C CNN
 F 1 "GND" H 5700 5080 30  0001 C CNN
 F 2 "" H 5700 5150 60  0001 C CNN
@@
 U 1 1 55D4CB6C
 P 3000 2500
-F 0 "PS1" H 3600 3600 60  0000 C CNN
-F 1 "PANSTAMP_NRG2" H 2600 3600 60  0000 C CNN
+F 0 "PS1" H 3000 3687 60  0000 C CNN
+F 1 "PANSTAMP_NRG2" H 3000 3581 60  0000 C CNN
 F 2 "mysmd:PANSTAMP_2" H 3050 2900 60  0001 C CNN
 F 3 "" H 3050 2900 60  0000 C CNN
@@
 $EndComp
 $Comp
-L VCC #PWR018
+L VCC #PWR017
 U 1 1 55D4CB73
 P 4150 2000
-F 0 "#PWR018" H 4150 2100 30  0001 C CNN
+F 0 "#PWR017" H 4150 2100 30  0001 C CNN
 F 1 "VCC" H 4150 2100 30  0000 C CNN
 F 2 "" H 4150 2000 60  0001 C CNN
@@
 $EndComp
 $Comp
-L GND #PWR019
+L GND #PWR018
 U 1 1 55D4CB79
 P 3000 3900
-F 0 "#PWR019" H 3000 3900 30  0001 C CNN
+F 0 "#PWR018" H 3000 3900 30  0001 C CNN
 F 1 "GND" H 3000 3830 30  0001 C CNN
 F 2 "" H 3000 3900 60  0001 C CNN
@@
 Text Label 1550 2700 0    60   ~ 0
 D5
-Text Label 1550 2900 0    60   ~ 0
+Text Label 1800 2900 0    60   ~ 0
 D3
 Text Label 1550 3000 0    60   ~ 0
@@
 Text Label 1550 2500 0    60   ~ 0
 D7
-Text Label 1550 2800 0    60   ~ 0
+Text Label 1800 2800 0    60   ~ 0
 D4
 Text Label 4400 1750 2    60   ~ 0
@@
 	4000 2700 4400 2700
 Wire Wire Line
-	4000 2800 4400 2800
-Wire Wire Line
-	4000 2900 4400 2900
-Wire Wire Line
-	4000 3000 4950 3000
-Wire Wire Line
-	4000 3100 4950 3100
-Wire Wire Line
-	4000 3200 4950 3200
-Wire Wire Line
 	2000 1600 1550 1600
 Wire Wire Line
@@
 	2000 2700 1550 2700
 Wire Wire Line
-	2000 2800 1550 2800
-Wire Wire Line
-	2000 2900 1550 2900
+	1250 2800 2000 2800
+Wire Wire Line
+	1250 2900 2000 2900
 Wire Wire Line
 	2000 3000 1550 3000
@@
 $EndComp
 $Comp
-L GND #PWR020
+L GND #PWR019
 U 1 1 55D4DC5B
 P 8200 1700
-F 0 "#PWR020" H 8200 1700 30  0001 C CNN
+F 0 "#PWR019" H 8200 1700 30  0001 C CNN
 F 1 "GND" H 8200 1630 30  0001 C CNN
 F 2 "" H 8200 1700 60  0001 C CNN
@@
 	8200 1700 8200 1650
 $Comp
-L VCC #PWR?
+L VCC #PWR020
 U 1 1 55D4C72B
 P 5150 6300
-F 0 "#PWR?" H 5150 6400 30  0001 C CNN
+F 0 "#PWR020" H 5150 6400 30  0001 C CNN
 F 1 "VCC" H 5150 6400 30  0000 C CNN
 F 2 "" H 5150 6300 60  0001 C CNN
@@
 	1    0    0    -1
 $EndComp
+Wire Wire Line
+	4000 3100 4400 3100
+Wire Wire Line
+	4000 3200 4400 3200
+Wire Wire Line
+	4000 3000 4400 3000
+$Comp
+L SW_PUSH SW1
+U 1 1 567B5528
+P 4700 2200
+F 0 "SW1" H 4700 2456 50  0000 C CNN
+F 1 "SW_PUSH" H 4700 2364 50  0000 C CNN
+F 2 "mysmd:switch-tact-noah" H 4700 2200 50  0001 C CNN
+F 3 "" H 4700 2200 50  0000 C CNN
+	1    4700 2200
+	-1   0    0    -1
+$EndComp
+$Comp
+L GND #PWR021
+U 1 1 567B560F
+P 5100 2300
+F 0 "#PWR021" H 5100 2300 30  0001 C CNN
+F 1 "GND" H 5100 2230 30  0001 C CNN
+F 2 "" H 5100 2300 60  0001 C CNN
+F 3 "" H 5100 2300 60  0001 C CNN
+	1    5100 2300
+	1    0    0    -1
+$EndComp
+Wire Wire Line
+	5000 2200 5100 2200
+Wire Wire Line
+	5100 2200 5100 2300
+Wire Wire Line
+	4000 2900 4950 2900
+Wire Wire Line
+	4000 2800 4400 2800
 $EndSCHEMATC
