File: cb-imu/cb-imu.kicad_pcb (KiCad board)
At the start: 4 copper layers, 25.4 x 56.6 mm, 31 parts, among them P1 CONN_01X14, P2 CONN_01X14, P3 CONN_01X02, U1 LSM9DS1, U2 ANTENNA, U3 MCP1702, U4 MMA8652FC

Commit message: PCB layout finished
Other:
- board text added: "+5V"
Changed lines of the file:
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@@
     (links 110)
     (no_connects 0)
-    (area 184.426859 44.579499 210.215481 101.570501)
+    (area 181.809499 44.579499 213.190501 102.472)
     (thickness 1.6002)
-    (drawings 75)
+    (drawings 79)
     (tracks 928)
     (zones 0)
@@
     (visible_elements FFFFF7BF)
     (pcbplotparams
-      (layerselection 0x010f0_80000001)
+      (layerselection 0x010f0_fffffff9)
       (usegerberextensions true)
       (excludeedgelayer true)
@@
     (descr "Through hole pin header")
     (tags "pin header")
-    (fp_text reference P3 (at 0.01 4.98 180) (layer F.SilkS)
+    (fp_text reference P3 (at 2.03 2.5 180) (layer F.SilkS)
       (effects (font (size 1 1) (thickness 0.15)))
     )
@@
       (xy 13.208 5.2324)) (layer F.SilkS) (width 0.00254))
   )
+  (gr_text GND (at 208.08 99.43 90) (layer B.SilkS)
+    (effects (font (size 1.27 1.016) (thickness 0.1524)) (justify mirror))
+  )
+  (gr_text +5V (at 200.8 99.16 90) (layer B.SilkS)
+    (effects (font (size 1.27 1.016) (thickness 0.1524)) (justify mirror))
+  )
+  (gr_text +5V (at 200.72 99.36 90) (layer F.SilkS)
+    (effects (font (size 1.27 1.016) (thickness 0.1524)))
+  )
+  (gr_text GND (at 208.1 99.46 90) (layer F.SilkS)
+    (effects (font (size 1.27 1.016) (thickness 0.1524)))
+  )
   (gr_line (start 212 46) (end 183 46) (angle 90) (layer Dwgs.User) (width 0.381))
