File: cb-linkit/cb-linkit.kicad_pcb (KiCad board)
At the start: 4 copper layers, 81 x 76 mm, 44 parts, among them P1 CONN_01X14, P2 CONN_01X14, P3 CONN_01X14, P4 CONN_01X14, P5 CONN_01X02, Q1 Q_NPN_EBC, Q2 Q_NPN_EBC, U1 Linkit_Smart_7688, U2 AP2114H-3.3, U6 SIM800L_module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

Commit message: Layout redone
Parts:
- removed the 1PIN at (119.6, 22.0)
- removed the 1PIN at (181.6, 89.0)
- removed ANT1: ANTENNA, myconnectors:SMA_RightAngle_Tyco
- removed the P3 at (164.6, 130.7)
- removed PS1: PANSTAMP_NRG2, mysmd:PANSTAMP_2
- added G***: PANSTAMPLOGO, mymods:PANSTAMPLOGO, F.Cu at (170.3, 35.5)
- added P1: CONN_01X14, myconnectors:pin_array_1x14, F.Cu at (166.2, 53.2)
- added REF**: Symbol_OSHW-Logo_SilkScreen, Symbols:Symbol_OSHW-Logo_SilkScreen, F.Cu at (117.5, 78.6)
- added REF**: Symbol_OSHW-Logo_SilkScreen_BIG, Symbols:Symbol_OSHW-Logo_SilkScreen_BIG, F.Cu at (177.9, 30.0)
- moved C21 185.4 mm to (174.4, 66.7), turned to 90 degrees
- moved D3 178.9 mm to (187.7, 81.8), turned to 90 degrees
- moved R17 178.2 mm to (173.5, 73.0), turned to 180 degrees
- moved C1 176.6 mm to (171.2, 66.7), turned to 90 degrees
- moved R16 174.9 mm to (174.3, 75.3), turned to 90 degrees
- moved U2 171.6 mm to (180.6, 67.4), turned to 270 degrees
- moved C12 171.6 mm to (176.0, 75.4), turned to 90 degrees
- moved C22 164.0 mm to (172.8, 66.7), turned to 90 degrees
- moved P5 160.7 mm to (179.7, 87.1), turned to 90 degrees
- moved C19 160.2 mm to (174.4, 70.5), turned to 270 degrees
- moved C10 159.4 mm to (181.6, 76.6)
- moved C20 156.6 mm to (172.8, 70.5), turned to 270 degrees
- moved R11 156.4 mm to (140.8, 44.1)
- moved PS2 149.6 mm to (123.5, 39.0)
- moved U8 141.6 mm to (172.1, 77.4), turned to 90 degrees
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- renumbered P1 to P3
Connections:
- P2 pad 11: Net-(P2-Pad11) -> PS1_RESET
- P2 pad 12: Net-(P2-Pad12) -> PS1_TEST
- P2 pad 13: Net-(P2-Pad13) -> GND
- P2 pad 14: GND -> +3V3
- P2 pad 8: Net-(P2-Pad8) -> PS1_RXD
- P2 pad 9: Net-(P2-Pad9) -> PS1_TXD
- P4 pad 14: VCC -> +3V3
- PS2 pad 13: VCC -> +3V3
- U1 pad 21: PS1_TEST -> PS1_RESET
- U1 pad 22: PS1_RESET -> PS1_TEST
- U1 pad 23: PS2_TEST -> PS2_RESET
- U1 pad 24: PS2_RESET -> PS2_TEST
Routing:
- net GND: track 0.00 -> 1215.9 mm, vias 0 -> 402
- net +3V3: track 0.00 -> 133.1 mm, vias 0 -> 1
- net +5V: track 0.00 -> 97.7 mm
- net PS2_TXD: track 0.00 -> 70.9 mm, vias 0 -> 3
- net PS2_TEST: track 0.00 -> 68.1 mm, vias 0 -> 4
- net PS2_RESET: track 0.00 -> 58.8 mm, vias 0 -> 4
- net PS2_RXD: track 0.00 -> 57.1 mm
- net Net-(R11-Pad2): track 0.00 -> 54.1 mm, vias 0 -> 6
- net Net-(R12-Pad2): track 0.00 -> 48.7 mm, vias 0 -> 6
- net PS1_TXD: track 0.00 -> 47.3 mm
- net PS1_RXD: track 0.00 -> 42.6 mm, vias 0 -> 2
- net PS1_TEST: track 0.00 -> 35.7 mm
- net Net-(R10-Pad2): track 0.00 -> 35.4 mm
- net PS1_RESET: track 0.00 -> 27.2 mm
- net VAA: track 0.00 -> 26.6 mm
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- added copper zone on B.Cu, net GND
- added copper zone on F.Cu, net GND
Other:
- board text added: "LIBREnet gateway 1.0"
- board text added: "Linkit Smart 7688"
- board text removed: "flex-board 1.0"

Commit message: Version 0.1 released
Other:
- board text added: "LIBREnet gateway 0.1"
- board text removed: "LIBREnet gateway 1.0"
Changed lines of the file:
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@@
-(kicad_pcb (version 4) (host pcbnew 0.201603021449+6606~42~ubuntu14.04.1-product)
+(kicad_pcb (version 4) (host pcbnew 0.201603031449+6606~43~ubuntu14.04.1-product)
   (general
     (links 86)
@@
     (title "Linkit carrier board")
     (date 2016-03-02)
-    (rev 1.0)
+    (rev 0.1)
     (company "panStamp (www.panstamp.com)")
   )
@@
   )
   (setup
-    (last_trace_width 0.762)
+    (last_trace_width 0.1524)
     (user_trace_width 0.1524)
     (user_trace_width 0.254)
@@
     (visible_elements FFFFF7BF)
     (pcbplotparams
-      (layerselection 0x010e0_fffffff9)
+      (layerselection 0x00020_7ffffff8)
       (usegerberextensions true)
       (excludeedgelayer true)
@@
   (gr_arc (start 114.58 21.96) (end 110.09 21.96) (angle 90) (layer Edge.Cuts) (width 0.381))
   (gr_arc (start 114.58 88.96) (end 114.58 93.48) (angle 90) (layer Edge.Cuts) (width 0.381))
-  (gr_text "LIBREnet gateway\n1.0" (at 123.33 75.44) (layer F.SilkS)
+  (gr_text "LIBREnet gateway\n0.1" (at 123.33 75.44) (layer F.SilkS)
     (effects (font (size 1.778 1.524) (thickness 0.1778)))
   )
