File: cb-linkit/cb-linkit.sch (KiCad schematic (older format))
At the start: 13 parts, among them Q1 Q_NPN_EBC, Q2 Q_NPN_EBC, U1 Linkit_Smart_7688, U6 SIM800L_module

Commit message: Layout redone
Connections:
- net PS1_RESET: now also U1.21 (GPIO16); no longer U1.22 (GPIO17)
- net PS1_TEST: now also U1.22 (GPIO17); no longer U1.21 (GPIO16)
- net PS2_RESET: now also U1.23 (GPIO19); no longer U1.24 (GPIO18)
- net PS2_TEST: now also U1.24 (GPIO18); no longer U1.23 (GPIO19)
Changed lines of the file:
@@
 Wire Wire Line
 	4550 1900 4400 1900
-Text GLabel 4550 3200 2    60   Input ~ 0
+Text GLabel 4550 3100 2    60   Input ~ 0
 PS1_TEST
 Wire Wire Line
 	4550 3200 4400 3200
-Text GLabel 4550 3100 2    60   Input ~ 0
+Text GLabel 4550 3200 2    60   Input ~ 0
 PS1_RESET
 Wire Wire Line
 	4550 3100 4400 3100
-Text GLabel 4550 3000 2    60   Input ~ 0
+Text GLabel 4550 2900 2    60   Input ~ 0
 PS2_TEST
 Wire Wire Line
 	4550 3000 4400 3000
-Text GLabel 4550 2900 2    60   Input ~ 0
+Text GLabel 4550 3000 2    60   Input ~ 0
 PS2_RESET
 Wire Wire Line
@@
 Wire Wire Line
 	7200 1800 7200 1850
-$Comp
-L +3V3 #PWR06
-U 1 1 56D72B7C
-P 7200 1800
-F 0 "#PWR06" H 7200 1650 50  0001 C CNN
-F 1 "+3V3" H 7218 1974 50  0000 C CNN
-F 2 "" H 7200 1800 50  0000 C CNN
-F 3 "" H 7200 1800 50  0000 C CNN
-	1    7200 1800
-	1    0    0    -1
-$EndComp
 Wire Wire Line
 	2950 3300 2400 3300
@@
 $EndComp
 $Comp
-L GND #PWR07
+L GND #PWR06
 U 1 1 56D72F77
 P 8950 3250
-F 0 "#PWR07" H 8950 3250 30  0001 C CNN
+F 0 "#PWR06" H 8950 3250 30  0001 C CNN
 F 1 "GND" H 8950 3180 30  0001 C CNN
 F 2 "" H 8950 3250 60  0001 C CNN
@@
 Wire Wire Line
 	8950 1800 8950 1850
+Wire Wire Line
+	8250 2850 7900 2850
+Text Label 7900 2850 0    60   ~ 0
+LED2
 $Comp
-L +3V3 #PWR08
-U 1 1 56D72F86
+L +3V3 #PWR?
+U 1 1 56D8716B
+P 7200 1800
+F 0 "#PWR?" H 7200 1650 50  0001 C CNN
+F 1 "+3V3" H 7218 1974 50  0000 C CNN
+F 2 "" H 7200 1800 50  0000 C CNN
+F 3 "" H 7200 1800 50  0000 C CNN
+	1    7200 1800
+	1    0    0    -1
+$EndComp
+$Comp
+L +3V3 #PWR?
+U 1 1 56D8724D
 P 8950 1800
-F 0 "#PWR08" H 8950 1650 50  0001 C CNN
+F 0 "#PWR?" H 8950 1650 50  0001 C CNN
 F 1 "+3V3" H 8968 1974 50  0000 C CNN
 F 2 "" H 8950 1800 50  0000 C CNN
@@
 	1    0    0    -1
 $EndComp
-Wire Wire Line
-	8250 2850 7900 2850
-Text Label 7900 2850 0    60   ~ 0
-LED2
 $EndSCHEMATC
