File: cb-linkit/rf.sch (KiCad schematic (older format))
At the start: 8 parts, among them P1 CONN_01X14, P2 CONN_01X14, P3 CONN_01X14, P4 CONN_01X14

Commit message: Layout redone
Parts:
- removed ANT1: ANTENNA, myconnectors:SMA_RightAngle_Tyco, symbol ANTENNA
- removed PS1: PANSTAMP_NRG2, mysmd:PANSTAMP_2, symbol PANSTAMP_NRG2-RESCUE-cb_co2
- renumbered P3 to P2, P2 to P3
Connections:
- net VCC renamed +3V3
- no-connect marks 84 -> 63
Changed lines of the file:
@@
 $EndDescr
-$Comp
-L GND #PWR028
-U 1 1 56D57026
-P 3500 3350
-F 0 "#PWR028" H 3500 3350 30  0001 C CNN
-F 1 "GND" H 3500 3280 30  0001 C CNN
-F 2 "" H 3500 3350 60  0001 C CNN
-F 3 "" H 3500 3350 60  0001 C CNN
-	1    3500 3350
-	-1   0    0    -1
-$EndComp
-$Comp
-L VCC #PWR029
-U 1 1 56D5702C
-P 4600 1500
-F 0 "#PWR029" H 4600 1600 30  0001 C CNN
-F 1 "VCC" H 4600 1600 30  0000 C CNN
-F 2 "" H 4600 1500 60  0000 C CNN
-F 3 "" H 4600 1500 60  0000 C CNN
-	1    4600 1500
-	1    0    0    -1
-$EndComp
-$Comp
-L PANSTAMP_NRG2-RESCUE-cb_co2 PS1
-U 1 1 56D57032
-P 3500 2000
-F 0 "PS1" H 4100 3100 60  0000 C CNN
-F 1 "PANSTAMP_NRG2" H 3100 3100 60  0000 C CNN
-F 2 "mysmd:PANSTAMP_2" H 3550 2400 60  0001 C CNN
-F 3 "" H 3550 2400 60  0000 C CNN
-	1    3500 2000
-	1    0    0    -1
-$EndComp
-$Comp
-L ANTENNA ANT1
-U 1 1 56D5706A
-P 5700 1350
-F 0 "ANT1" H 6128 1553 60  0000 L CNN
-F 1 "ANTENNA" H 6128 1447 60  0000 L CNN
-F 2 "myconnectors:SMA_RightAngle_Tyco" H 5700 1350 60  0001 C CNN
-F 3 "" H 5700 1350 60  0000 C CNN
-	1    5700 1350
-	1    0    0    -1
-$EndComp
-Wire Wire Line
-	4600 1600 4600 1500
-Wire Wire Line
-	4500 1600 4600 1600
-Wire Wire Line
-	3200 3250 3200 3300
-Wire Wire Line
-	3200 3300 3800 3300
-Wire Wire Line
-	3800 3300 3800 3250
-Wire Wire Line
-	3700 3250 3700 3300
-Connection ~ 3700 3300
-Wire Wire Line
-	3600 3250 3600 3300
-Connection ~ 3600 3300
-Wire Wire Line
-	3500 3250 3500 3350
-Connection ~ 3500 3300
-Wire Wire Line
-	3400 3250 3400 3300
-Connection ~ 3400 3300
-Wire Wire Line
-	3300 3250 3300 3300
-Connection ~ 3300 3300
 $Comp
 L CONN_01X14 P1
@@
 $EndComp
 $Comp
-L CONN_01X14 P3
+L CONN_01X14 P2
 U 1 1 56D574EA
 P 7550 2300
-F 0 "P3" H 7550 3050 50  0000 C CNN
+F 0 "P2" H 7550 3050 50  0000 C CNN
 F 1 "CONN_01X14" V 7650 2300 50  0000 C CNN
 F 2 "Pin_Headers:Pin_Header_Straight_1x14" H 7550 2300 60  0001 C CNN
@@
 	-1   0    0    -1
 $EndComp
-Text Label 8250 2750 2    60   ~ 0
-PS1_TEST
-Text Label 8250 2650 2    60   ~ 0
-PS1_RESET
-$Comp
-L VCC #PWR030
-U 1 1 56D574FD
-P 7900 3050
-F 0 "#PWR030" H 7900 3150 30  0001 C CNN
-F 1 "VCC" H 7900 3150 30  0000 C CNN
-F 2 "" H 7900 3050 60  0001 C CNN
-F 3 "" H 7900 3050 60  0001 C CNN
-	1    7900 3050
-	-1   0    0    1
-$EndComp
-Text Label 8250 2350 2    60   ~ 0
-PS1_RXD
-Text Label 8250 2450 2    60   ~ 0
-PS1_TXD
-$Comp
-L GND #PWR031
+$Comp
+L GND #PWR028
 U 1 1 56D5750D
 P 6850 3050
-F 0 "#PWR031" H 6850 3050 30  0001 C CNN
+F 0 "#PWR028" H 6850 3050 30  0001 C CNN
 F 1 "GND" H 6850 2980 30  0001 C CNN
 F 2 "" H 6850 3050 60  0001 C CNN
@@
 $EndComp
 $Comp
-L GND #PWR032
+L GND #PWR029
 U 1 1 56D57516
 P 8100 3050
-F 0 "#PWR032" H 8100 3050 30  0001 C CNN
+F 0 "#PWR029" H 8100 3050 30  0001 C CNN
 F 1 "GND" H 8100 2980 30  0001 C CNN
 F 2 "" H 8100 3050 60  0001 C CNN
@@
 NoConn ~ 6950 2750
 NoConn ~ 6950 2850
-Wire Wire Line
-	4500 1250 5250 1250
-$Comp
-L GND #PWR033
-U 1 1 56D6C6A4
-P 5150 1450
-F 0 "#PWR033" H 5150 1450 30  0001 C CNN
-F 1 "GND" H 5150 1380 30  0001 C CNN
-F 2 "" H 5150 1450 60  0001 C CNN
-F 3 "" H 5150 1450 60  0001 C CNN
-	1    5150 1450
-	0    1    -1   0
-$EndComp
-Wire Wire Line
-	5250 1450 5150 1450
-NoConn ~ 2500 2700
-NoConn ~ 2500 2600
-NoConn ~ 2500 2500
-NoConn ~ 2500 2400
-NoConn ~ 2500 2300
-NoConn ~ 2500 2000
-NoConn ~ 2500 1800
-NoConn ~ 2500 1700
-NoConn ~ 2500 1600
-NoConn ~ 2500 1500
-NoConn ~ 2500 1400
-NoConn ~ 2500 1300
-NoConn ~ 2500 1200
-NoConn ~ 2500 1100
-NoConn ~ 4500 2700
-NoConn ~ 4500 2600
-NoConn ~ 4500 2500
-NoConn ~ 4500 2400
-NoConn ~ 4500 2300
-NoConn ~ 4500 2200
-NoConn ~ 4500 2100
-Text GLabel 2300 2100 0    60   Input ~ 0
+Text GLabel 8250 2450 2    60   Input ~ 0
 PS1_TXD
-Text GLabel 2300 2200 0    60   Input ~ 0
+Text GLabel 8250 2350 2    60   Input ~ 0
 PS1_RXD
-Wire Wire Line
-	2500 2100 2300 2100
-Wire Wire Line
-	2500 2200 2300 2200
-Text GLabel 4600 1800 2    60   Input ~ 0
+Text GLabel 8250 2750 2    60   Input ~ 0
 PS1_TEST
-Wire Wire Line
-	4500 1800 4600 1800
-Text GLabel 4600 1700 2    60   Input ~ 0
+Text GLabel 8250 2650 2    60   Input ~ 0
 PS1_RESET
-Wire Wire Line
-	4500 1700 4600 1700
-$Comp
-L GND #PWR034
+$Comp
+L GND #PWR030
 U 1 1 56D6D450
 P 3500 6300
-F 0 "#PWR034" H 3500 6300 30  0001 C CNN
+F 0 "#PWR030" H 3500 6300 30  0001 C CNN
 F 1 "GND" H 3500 6230 30  0001 C CNN
 F 2 "" H 3500 6300 60  0001 C CNN
@@
 	1    3500 6300
 	-1   0    0    -1
-$EndComp
-$Comp
-L VCC #PWR035
-U 1 1 56D6D456
-P 4600 4450
-F 0 "#PWR035" H 4600 4550 30  0001 C CNN
-F 1 "VCC" H 4600 4550 30  0000 C CNN
-F 2 "" H 4600 4450 60  0000 C CNN
-F 3 "" H 4600 4450 60  0000 C CNN
-	1    4600 4450
-	1    0    0    -1
 $EndComp
 $Comp
@@
 Connection ~ 3300 6250
 $Comp
-L CONN_01X14 P2
+L CONN_01X14 P3
 U 1 1 56D6D477
 P 7150 5250
-F 0 "P2" H 7150 6000 50  0000 C CNN
+F 0 "P3" H 7150 6000 50  0000 C CNN
 F 1 "CONN_01X14" V 7250 5250 50  0000 C CNN
 F 2 "Pin_Headers:Pin_Header_Straight_1x14" H 7150 5250 60  0001 C CNN
@@
 Text Label 8250 5600 2    60   ~ 0
 PS2_RESET
-$Comp
-L VCC #PWR036
-U 1 1 56D6D485
-P 7900 6000
-F 0 "#PWR036" H 7900 6100 30  0001 C CNN
-F 1 "VCC" H 7900 6100 30  0000 C CNN
-F 2 "" H 7900 6000 60  0001 C CNN
-F 3 "" H 7900 6000 60  0001 C CNN
-	1    7900 6000
-	-1   0    0    1
-$EndComp
 Text Label 8250 5300 2    60   ~ 0
 PS2_RXD
@@
 PS2_TXD
 $Comp
-L GND #PWR037
+L GND #PWR031
 U 1 1 56D6D48D
 P 6850 6000
-F 0 "#PWR037" H 6850 6000 30  0001 C CNN
+F 0 "#PWR031" H 6850 6000 30  0001 C CNN
 F 1 "GND" H 6850 5930 30  0001 C CNN
 F 2 "" H 6850 6000 60  0001 C CNN
@@
 $EndComp
 $Comp
-L GND #PWR038
+L GND #PWR032
 U 1 1 56D6D493
 P 8100 6000
-F 0 "#PWR038" H 8100 6000 30  0001 C CNN
+F 0 "#PWR032" H 8100 6000 30  0001 C CNN
 F 1 "GND" H 8100 5930 30  0001 C CNN
 F 2 "" H 8100 6000 60  0001 C CNN
@@
 	4500 4200 5250 4200
 $Comp
-L GND #PWR039
+L GND #PWR033
 U 1 1 56D6D4B9
 P 5150 4400
-F 0 "#PWR039" H 5150 4400 30  0001 C CNN
+F 0 "#PWR033" H 5150 4400 30  0001 C CNN
 F 1 "GND" H 5150 4330 30  0001 C CNN
 F 2 "" H 5150 4400 60  0001 C CNN
@@
 Wire Wire Line
 	4500 4650 4600 4650
+$Comp
+L +3V3 #PWR034
+U 1 1 56D7678E
+P 4600 4450
+F 0 "#PWR034" H 4600 4300 50  0001 C CNN
+F 1 "+3V3" H 4618 4624 50  0000 C CNN
+F 2 "" H 4600 4450 50  0000 C CNN
+F 3 "" H 4600 4450 50  0000 C CNN
+	1    4600 4450
+	1    0    0    -1
+$EndComp
+$Comp
+L +3V3 #PWR035
+U 1 1 56D76A8C
+P 7900 6000
+F 0 "#PWR035" H 7900 5850 50  0001 C CNN
+F 1 "+3V3" H 7918 6174 50  0000 C CNN
+F 2 "" H 7900 6000 50  0000 C CNN
+F 3 "" H 7900 6000 50  0000 C CNN
+	1    7900 6000
+	-1   0    0    1
+$EndComp
+$Comp
+L +3V3 #PWR036
+U 1 1 56D76ADE
+P 7900 3050
+F 0 "#PWR036" H 7900 2900 50  0001 C CNN
+F 1 "+3V3" H 7918 3224 50  0000 C CNN
+F 2 "" H 7900 3050 50  0000 C CNN
+F 3 "" H 7900 3050 50  0000 C CNN
+	1    7900 3050
+	-1   0    0    1
+$EndComp
 $EndSCHEMATC
