File: cb-minibat/cb-minibat.sch (KiCad schematic (older format))
At the start: 37 parts, among them P1 CONN_01X14, P2 CONN_01X14, P3 CONN_8, SW1 SW_PUSH, U1 BMP180, U2 MAX1724, U3 SI7021, U4 M74VHC1GT08, U5 MCP1702, U6 LSM9DS0

Commit message: Title fixed and schematic created in PDF format
Parts:
- D1: symbol D -> D-RESCUE-cb-minibat
Changed lines of the file:
@@
 EESchema Schematic File Version 2
+LIBS:cb-minibat-rescue
 LIBS:power
 LIBS:device
@@
 LIBS:memory
 LIBS:xilinx
-LIBS:special
 LIBS:microcontrollers
 LIBS:dsp
@@
 encoding utf-8
 Sheet 1 1
-Title "Clima sensor board for panStamp"
+Title "Minibat sensor board for panStamp"
 Date "17 Mar 2015"
 Rev "1.0"
@@
 TOANT
 $Comp
-L D D1
+L D-RESCUE-cb-minibat D1
 U 1 1 55474E1B
 P 3800 7000

Commit message: Adding MMA8652 accelerometer and PCB meander antenna
Parts:
- removed ANT1: ANTENNA, myconnectors:SMA_RightAngle_Tyco, symbol ANTENNA
- removed ANT2: ANTENNA, myconnectors:U.FL_CONN, symbol ANTENNA
- removed C10: 3.9p, mysmd:SM0603S, symbol C
- removed C11: 0.3p, mysmd:SM0603S, symbol C
- removed C12: 4.7u, mysmd:SM0603S, symbol C
- removed C13: 220n, mysmd:SM0603S, symbol C
- removed C14, C9: 10u, mysmd:SM0603S, symbol C
- removed C15: 100n, mysmd:SM0603S, symbol C
- removed D1: SD0603S040S0R2, mysmd:SM0603S, symbol D-RESCUE-cb-minibat
- removed L2: 18n, mysmd:SM0603S, symbol INDUCTOR
- removed L3: ANTENNA, 0868AT43A0020, symbol INDUCTOR
- removed P3: CONN_8, myconnectors:PIN_ARRAY_8X1, symbol CONN_01X08
- removed R1: 0, mysmd:SM0603S, symbol R
- removed U2: MAX1724, libcms:SOT23_6, symbol MAX1724
- removed U4: M74VHC1GT08, libcms:SOT23-5, symbol M74VHC1GT08
- removed U5: MCP1702, libcms:SOT23, symbol MCP1702
- removed U6: LSM9DS0, mysmd:LGA24, symbol LSM9DS0
- added U2: MMA8652FC, mysmd:DFN-10, symbol MMA8652FC
- added U4: ANTENNA, myconnectors:U.FL_CONN, symbol ANTENNA
- C1: value 10u -> 100n
- C4: value 10u -> 1u
- C5: value 1u -> 100n
- C6, C7: value 100n -> N.P.
- L1: value 4.7u -> 0; footprint libcms:SM0805 -> mysmd:SM0603S
- PS1: symbol PANSTAMP_NRG2 -> PANSTAMP_NRG2-RESCUE-cb-minibat
Connections:
- net +5V is gone; now on an unnamed net: C7.1
- net D16: now also C4.1, C5.1, U2.1 (VDD), U2.8 (VDDIO)
- net D8: now also U2.5 (INT2)
- net D9: now also U2.3 (INT1)
- net GND: now also SW1.1, U2.6 (GND), U2.7 (GND), U2.9 (GND), U4.2 (GND); no longer SW1.2
- net I2C_SCL: now also U2.2 (SCL)
- net I2C_SDA: now also U2.10 (SDA)
- net RESET: now also SW1.2; no longer SW1.1
- net TOANT: now also C6.1, L1.1, U4.1 (RF)
- net VCC: no longer C4.1, C5.1, C6.1
- net +BATT: no longer names the net of C1.1
- net +BATT: now also U2.4 (BYP); no longer L1.1
- no-connect marks 2 -> 0
