File: cb-minibat/cb-minibat.sch (KiCad schematic (older format))
At the start: 21 parts, among them P1 CONN_01X14, P2 CONN_01X14, SW1 SW_PUSH, U1 BMP180, U2 MMA8652FC, U3 SI7021, U4 ANTENNA

Commit message: New version 2.1 with support for BME680
Parts:
- removed U1: BMP180, mysmd:BMP180, symbol BMP180
- added U1: BME680, mysmd:BME680, symbol BME680
Connections:
- net GND: now also U1.1 (GND), U1.5 (ADDR), U1.7 (GND)
- net I2C_SCL: now also U1.4 (SCL)
- net I2C_SDA: now also U1.3 (SDA)
- net VCC: now also U1.2 (VDDIO), U1.6 (VDDIO), U1.8 (VDD)
Other:
- moved on the sheet: C2, C3
Changed lines of the file:
@@
 LIBS:contrib
 LIBS:valves
-LIBS:atmega8
-LIBS:atmel89cxxxx
-LIBS:atmel-1
-LIBS:atmel-2005
-LIBS:avr
-LIBS:avr-1
-LIBS:avr-2
-LIBS:avr-3
-LIBS:avr-4
-LIBS:hopf
-LIBS:rfm-ash
-LIBS:mycomponents
+LIBS:panstamp
 LIBS:cb-minibat-cache
 EELAYER 25 0
@@
 Sheet 1 1
 Title "Minibat sensor board for panStamp"
-Date "2016-06-07"
-Rev "2.0"
+Date "2017-11-14"
+Rev "2.1"
 Comp "www.panstamp.com"
 Comment1 ""
@@
 L C C2
 U 1 1 5508513D
-P 3650 4150
-F 0 "C2" H 3700 4250 50  0000 L CNN
-F 1 "1u" H 3700 4050 50  0000 L CNN
-F 2 "mysmd:SM0603S" H 3650 4150 60  0001 C CNN
-F 3 "" H 3650 4150 60  0001 C CNN
-	1    3650 4150
+P 3450 4200
+F 0 "C2" H 3500 4300 50  0000 L CNN
+F 1 "1u" H 3500 4100 50  0000 L CNN
+F 2 "mysmd:SM0603S" H 3450 4200 60  0001 C CNN
+F 3 "" H 3450 4200 60  0001 C CNN
+	1    3450 4200
 	1    0    0    -1
 $EndComp
@@
 L GND #PWR06
 U 1 1 5508513E
-P 3650 4400
-F 0 "#PWR06" H 3650 4400 30  0001 C CNN
-F 1 "GND" H 3650 4330 30  0001 C CNN
-F 2 "" H 3650 4400 60  0001 C CNN
-F 3 "" H 3650 4400 60  0001 C CNN
-	1    3650 4400
+P 3450 4450
+F 0 "#PWR06" H 3450 4450 30  0001 C CNN
+F 1 "GND" H 3450 4380 30  0001 C CNN
+F 2 "" H 3450 4450 60  0001 C CNN
+F 3 "" H 3450 4450 60  0001 C CNN
+	1    3450 4450
 	1    0    0    -1
 $EndComp
@@
 L C C3
 U 1 1 5508513F
-P 4050 4150
-F 0 "C3" H 4100 4250 50  0000 L CNN
-F 1 "100n" H 4100 4050 50  0000 L CNN
-F 2 "mysmd:SM0603S" H 4050 4150 60  0001 C CNN
-F 3 "" H 4050 4150 60  0001 C CNN
-	1    4050 4150
+P 3850 4200
+F 0 "C3" H 3900 4300 50  0000 L CNN
+F 1 "100n" H 3900 4100 50  0000 L CNN
+F 2 "mysmd:SM0603S" H 3850 4200 60  0001 C CNN
+F 3 "" H 3850 4200 60  0001 C CNN
+	1    3850 4200
 	1    0    0    -1
 $EndComp
@@
 L GND #PWR07
 U 1 1 55085140
-P 4050 4400
-F 0 "#PWR07" H 4050 4400 30  0001 C CNN
-F 1 "GND" H 4050 4330 30  0001 C CNN
-F 2 "" H 4050 4400 60  0001 C CNN
-F 3 "" H 4050 4400 60  0001 C CNN
-	1    4050 4400
+P 3850 4450
+F 0 "#PWR07" H 3850 4450 30  0001 C CNN
+F 1 "GND" H 3850 4380 30  0001 C CNN
+F 2 "" H 3850 4450 60  0001 C CNN
+F 3 "" H 3850 4450 60  0001 C CNN
+	1    3850 4450
 	1    0    0    -1
 $EndComp
@@
 L VCC #PWR09
 U 1 1 55085145
-P 3650 3900
-F 0 "#PWR09" H 3650 4000 30  0001 C CNN
-F 1 "VCC" H 3650 4000 30  0000 C CNN
-F 2 "" H 3650 3900 60  0001 C CNN
-F 3 "" H 3650 3900 60  0001 C CNN
-	1    3650 3900
+P 3450 3950
+F 0 "#PWR09" H 3450 4050 30  0001 C CNN
+F 1 "VCC" H 3450 4050 30  0000 C CNN
+F 2 "" H 3450 3950 60  0001 C CNN
+F 3 "" H 3450 3950 60  0001 C CNN
+	1    3450 3950
 	1    0    0    -1
 $EndComp
@@
 L VCC #PWR010
 U 1 1 55085146
-P 4050 3900
-F 0 "#PWR010" H 4050 4000 30  0001 C CNN
-F 1 "VCC" H 4050 4000 30  0000 C CNN
-F 2 "" H 4050 3900 60  0001 C CNN
-F 3 "" H 4050 3900 60  0001 C CNN
-	1    4050 3900
+P 3850 3950
+F 0 "#PWR010" H 3850 4050 30  0001 C CNN
+F 1 "VCC" H 3850 4050 30  0000 C CNN
+F 2 "" H 3850 3950 60  0001 C CNN
+F 3 "" H 3850 3950 60  0001 C CNN
+	1    3850 3950
 	1    0    0    -1
 $EndComp
@@
 D22
 $Comp
-L BMP180 U1
-U 1 1 5508514C
-P 1950 4250
-F 0 "U1" H 1750 4600 60  0000 C CNN
-F 1 "BMP180" H 1850 3900 60  0000 C CNN
-F 2 "mysmd:BMP180" H 1950 4250 60  0001 C CNN
-F 3 "" H 1950 4250 60  0000 C CNN
-	1    1950 4250
-	1    0    0    -1
-$EndComp
-$Comp
 L VCC #PWR015
 U 1 1 5508514D
-P 1250 3950
-F 0 "#PWR015" H 1250 4050 30  0001 C CNN
-F 1 "VCC" H 1250 4050 30  0000 C CNN
-F 2 "" H 1250 3950 60  0001 C CNN
-F 3 "" H 1250 3950 60  0001 C CNN
-	1    1250 3950
+P 1950 3650
+F 0 "#PWR015" H 1950 3750 30  0001 C CNN
+F 1 "VCC" H 1950 3750 30  0000 C CNN
+F 2 "" H 1950 3650 60  0001 C CNN
+F 3 "" H 1950 3650 60  0001 C CNN
+	1    1950 3650
 	1    0    0    -1
 $EndComp
@@
 L GND #PWR016
 U 1 1 5508514E
-P 1250 4500
-F 0 "#PWR016" H 1250 4500 30  0001 C CNN
-F 1 "GND" H 1250 4430 30  0001 C CNN
-F 2 "" H 1250 4500 60  0001 C CNN
-F 3 "" H 1250 4500 60  0001 C CNN
-	1    1250 4500
-	1    0    0    -1
-$EndComp
-Text Label 3050 4400 2    60   ~ 0
+P 1950 4800
+F 0 "#PWR016" H 1950 4800 30  0001 C CNN
+F 1 "GND" H 1950 4730 30  0001 C CNN
+F 2 "" H 1950 4800 60  0001 C CNN
+F 3 "" H 1950 4800 60  0001 C CNN
+	1    1950 4800
+	1    0    0    -1
+$EndComp
+Text Label 3000 4400 2    60   ~ 0
 I2C_SCL
-Text Label 3050 4100 2    60   ~ 0
+Text Label 3000 4050 2    60   ~ 0
 I2C_SDA
 Text Label 1000 1950 0    60   ~ 0
@@
 Connection ~ 5900 6500
 Wire Wire Line
-	3650 4300 3650 4400
-Wire Wire Line
-	3650 3900 3650 4000
-Wire Wire Line
-	4050 4300 4050 4400
-Wire Wire Line
-	4050 3900 4050 4000
+	3450 4350 3450 4450
+Wire Wire Line
+	3450 3950 3450 4050
+Wire Wire Line
+	3850 4350 3850 4450
+Wire Wire Line
+	3850 3950 3850 4050
 Wire Wire Line
 	4800 4250 4800 4500
@@
 	6600 4700 6600 4750
 Wire Wire Line
-	1350 4150 1250 4150
-Wire Wire Line
-	1250 4150 1250 3950
-Wire Wire Line
-	1350 4050 1250 4050
-Connection ~ 1250 4050
-Wire Wire Line
-	1350 4450 1250 4450
-Wire Wire Line
-	1250 4450 1250 4500
-Wire Wire Line
-	2600 4100 3050 4100
-Wire Wire Line
-	2600 4400 3050 4400
+	2550 4050 3000 4050
+Wire Wire Line
+	2550 4400 3000 4400
 Wire Wire Line
 	3450 1200 3850 1200
@@
 Wire Wire Line
 	7950 1250 9050 1250
+$Comp
+L BME680 U1
+U 1 1 5A0AB40D
+P 2050 4200
+F 0 "U1" H 1850 4500 60  0000 C CNN
+F 1 "BME680" H 1750 3800 60  0000 C CNN
+F 2 "mysmd:BME680" H 2150 4050 60  0001 C CNN
+F 3 "" H 2150 4050 60  0000 C CNN
+	1    2050 4200
+	-1   0    0    -1
+$EndComp
+Wire Wire Line
+	1850 4700 1850 4750
+Wire Wire Line
+	1850 4750 2050 4750
+Wire Wire Line
+	2050 4750 2050 4700
+Wire Wire Line
+	1950 4700 1950 4800
+Connection ~ 1950 4750
+Wire Wire Line
+	1850 3750 1850 3700
+Wire Wire Line
+	1850 3700 2050 3700
+Wire Wire Line
+	2050 3700 2050 3750
+Wire Wire Line
+	1950 3650 1950 3750
+Connection ~ 1950 3700
 $EndSCHEMATC
