File: cb-io1/cb-io.kicad_pcb (KiCad board)
At the start: 4 copper layers, 81 x 76 mm, 60 parts, among them P1 CONN_01X14, P10 CONN_01X03, P11 CONN_01X03, P2 CONN_01X14, P3 CONN_01X02, P4 CONN_01X02, P5 CONN_01X02, P7 CONN_01X03, P8 CONN_01X03, P9 CONN_01X03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

Commit message: Fixed orientation of D4
Parts:
- D4: footprint mysmd:SMA -> SMA
- turned D4 to 0 degrees
Changed lines of the file:
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@@
-(kicad_pcb (version 4) (host pcbnew 0.201603210401+6634~43~ubuntu14.04.1-product)
+(kicad_pcb (version 4) (host pcbnew 4.1.0-alpha+201605170746+6811~44~ubuntu14.04.1-product)
   (general
-    (links 140)
+    (links 0)
     (no_connects 0)
-    (area 191.671286 15.8538 275.923714 104.9886)
+    (area 192.679499 25.919499 274.090512 102.310501)
     (thickness 1.6002)
     (drawings 40)
@@
   )
   (setup
-    (last_trace_width 0.508)
+    (last_trace_width 0.1524)
     (user_trace_width 0.1524)
     (user_trace_width 0.2032)
@@
     (add_net VAA)
   )
+  (module SMA (layer Front)
+    (at 230.95 88.29)
+    (fp_text reference D4 (at 4.83 -0.08 90) (layer F.SilkS)
+      (effects (font (size 0.889 0.762) (thickness 0.1524)))
+    )
+    (fp_text value D_Schottky (at 0 2.159) (layer F.SilkS) hide
+      (effects (font (size 0.889 0.762) (thickness 0.1524)))
+    )
+    (fp_line (start 0.508 1.143) (end 0.508 -1.143) (layer F.SilkS) (width 0.381))
+    (fp_line (start 3.429 -1.27) (end 3.429 1.143) (layer F.SilkS) (width 0.381))
+    (fp_line (start -3.556 -1.27) (end 3.429 -1.27) (layer F.SilkS) (width 0.381))
+    (fp_line (start 3.429 -1.27) (end 3.81 -1.27) (layer F.SilkS) (width 0.381))
+    (fp_line (start 3.81 -1.27) (end 3.81 1.143) (layer F.SilkS) (width 0.381))
+    (fp_line (start 3.81 1.143) (end -3.81 1.143) (layer F.SilkS) (width 0.381))
+    (fp_line (start -3.81 1.143) (end -3.81 -1.27) (layer F.SilkS) (width 0.381))
+    (pad 2 smd rect (at -1.99898 0) (size 2.50952 1.70942) (layers Front F.Paste F.Mask)
+      (net 18 "Net-(D4-Pad2)"))
+    (pad 1 smd rect (at 1.99898 0) (size 2.50952 1.70942) (layers Front F.Paste F.Mask)
+      (net 10 VAA))
+  )
   (module myconnectors:pin_array_1x14 (layer Front)
     (at 206.00322 61.88308 270)
@@
   (module mymods:BAT_AA_HOLDER_02 (layer Front)
     (at 251.9 88.6 270)
-    (fp_text reference BT1 (at -50.86 -12.99 360) (layer F.SilkS)
+    (fp_text reference BT1 (at -50.86 -12.99) (layer F.SilkS)
       (effects (font (thickness 0.3048)))
     )
@@
   (module mysmd:SOD323 (layer Front)
     (at 217.08 87.27 270)
-    (fp_text reference D3 (at -2.47 0.83 360) (layer F.SilkS)
+    (fp_text reference D3 (at -2.47 0.83) (layer F.SilkS)
       (effects (font (size 0.889 0.762) (thickness 0.1524)))
     )
@@
       (net 10 VAA))
   )
-  (module mysmd:SMA (layer Front)
-    (at 230.95 88.29 180)
-    (fp_text reference D4 (at 4.83 -0.08 270) (layer F.SilkS)
-      (effects (font (size 0.889 0.762) (thickness 0.1524)))
-    )
-    (fp_text value D_Schottky (at 0 2.159 180) (layer F.SilkS) hide
-      (effects (font (size 0.889 0.762) (thickness 0.1524)))
-    )
-    (fp_line (start 0.508 1.143) (end 0.508 -1.143) (layer F.SilkS) (width 0.381))
-    (fp_line (start 3.429 -1.27) (end 3.429 1.143) (layer F.SilkS) (width 0.381))
-    (fp_line (start -3.556 -1.27) (end 3.429 -1.27) (layer F.SilkS) (width 0.381))
-    (fp_line (start 3.429 -1.27) (end 3.81 -1.27) (layer F.SilkS) (width 0.381))
-    (fp_line (start 3.81 -1.27) (end 3.81 1.143) (layer F.SilkS) (width 0.381))
-    (fp_line (start 3.81 1.143) (end -3.81 1.143) (layer F.SilkS) (width 0.381))
-    (fp_line (start -3.81 1.143) (end -3.81 -1.27) (layer F.SilkS) (width 0.381))
-    (pad 1 smd rect (at -1.99898 0 180) (size 2.50952 1.70942) (layers Front F.Paste F.Mask)
-      (net 10 VAA))
-    (pad 2 smd rect (at 1.99898 0 180) (size 2.50952 1.70942) (layers Front F.Paste F.Mask)
-      (net 18 "Net-(D4-Pad2)"))
-  )
   (module mysmd:SOD323 (layer Front)
     (at 210.41 87.27 270)
-    (fp_text reference D5 (at -2.52 0.01 360) (layer F.SilkS)
+    (fp_text reference D5 (at -2.52 0.01) (layer F.SilkS)
       (effects (font (size 0.889 0.762) (thickness 0.1524)))
     )
@@
     (at 231.25 84 270)
     (tags SOT23)
-    (fp_text reference U1 (at -2.15 -0.02 360) (layer F.SilkS)
+    (fp_text reference U1 (at -2.15 -0.02) (layer F.SilkS)
       (effects (font (size 0.762 0.762) (thickness 0.11938)))
     )
@@
     (at 220.23 87.23 180)
     (tags SOT23)
-    (fp_text reference Q1 (at -2.48 0.5 360) (layer F.SilkS)
+    (fp_text reference Q1 (at -2.48 0.5) (layer F.SilkS)
       (effects (font (size 0.762 0.762) (thickness 0.11938)))
     )
@@
     (at 213.58 87.23 180)
     (tags SOT23)
-    (fp_text reference Q2 (at 0.02 2.5 360) (layer F.SilkS)
+    (fp_text reference Q2 (at 0.02 2.5) (layer F.SilkS)
       (effects (font (size 0.762 0.762) (thickness 0.11938)))
     )
@@
     (tags "CMS SOT")
     (attr smd)
-    (fp_text reference D7 (at -2.18 -0.39 360) (layer F.SilkS)
+    (fp_text reference D7 (at -2.18 -0.39) (layer F.SilkS)
       (effects (font (size 0.762 0.762) (thickness 0.1905)))
     )
@@
     (tags "CMS SOT")
     (attr smd)
-    (fp_text reference D8 (at -2.24 0.02 360) (layer F.SilkS)
+    (fp_text reference D8 (at -2.24 0.02) (layer F.SilkS)
       (effects (font (size 0.762 0.762) (thickness 0.1905)))
     )
@@
     (tags "CMS SOT")
     (attr smd)
-    (fp_text reference D9 (at -2.22 0 360) (layer F.SilkS)
+    (fp_text reference D9 (at -2.22 0) (layer F.SilkS)
       (effects (font (size 0.762 0.762) (thickness 0.1905)))
     )
@@
     (tags "CMS SOT")
     (attr smd)
-    (fp_text reference D10 (at -2.23 -0.02 360) (layer F.SilkS)
+    (fp_text reference D10 (at -2.23 -0.02) (layer F.SilkS)
       (effects (font (size 0.762 0.762) (thickness 0.1905)))
     )
@@
     (tags "CMS SOT")
     (attr smd)
-    (fp_text reference D11 (at -2.32 -0.03 360) (layer F.SilkS)
+    (fp_text reference D11 (at -2.32 -0.03) (layer F.SilkS)
       (effects (font (size 0.762 0.762) (thickness 0.1905)))
     )
@@
     (descr "Through hole pin header")
     (tags "pin header")
-    (fp_text reference JP1 (at -0.08 4.82 360) (layer F.SilkS)
+    (fp_text reference JP1 (at -0.08 4.82) (layer F.SilkS)
       (effects (font (size 1 1) (thickness 0.15)))
     )
@@
     (descr "Through hole pin header")
     (tags "pin header")
-    (fp_text reference D12 (at -2.5 1.25 360) (layer F.SilkS)
+    (fp_text reference D12 (at -2.5 1.25) (layer F.SilkS)
       (effects (font (size 1 1) (thickness 0.15)))
     )
@@
     (descr "Through hole pin header")
     (tags "pin header")
-    (fp_text reference D13 (at -2.5 1 360) (layer F.SilkS)
+    (fp_text reference D13 (at -2.5 1) (layer F.SilkS)
       (effects (font (size 1 1) (thickness 0.15)))
     )
