File: cb-esp/cb-esp.kicad_pcb (KiCad board)
At the start: 4 copper layers, 25.4 x 55.8 mm, 24 parts, among them P1 CONN_01X07, P2 CONN_01X07, P3 CONN_01X02, SW1 SW_PUSH_SMALL, SW2 SW_PUSH_SMALL, U1 MCP1702, U2 ESP-12E, U3 LY-SK10

Commit message: Small changes
Other:
- board text added: "wifiStick 1.0"
- board text removed: "uStation 1.0"
Changed lines of the file:
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@@
     (effects (font (size 1.27 1.016) (thickness 0.1778)))
   )
-  (gr_text "uStation\n1.0" (at 124.968 106.68) (layer F.SilkS)
+  (gr_text "wifiStick\n1.0" (at 124.968 106.68) (layer F.SilkS)
     (effects (font (size 1.27 1.143) (thickness 0.1524)))
   )

Commit message: Board renamed to espStick
Other:
- board text added: "espStick 1.0"
- board text removed: "wifiStick 1.0"
Changed lines of the file:
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@@
-(kicad_pcb (version 4) (host pcbnew 0.201511131146+6311~30~ubuntu14.04.1-product)
+(kicad_pcb (version 4) (host pcbnew 0.201512201246+6385~39~ubuntu14.04.1-stable)
   (general
     (links 58)
@@
     (effects (font (size 1.27 1.016) (thickness 0.1778)))
   )
-  (gr_text "wifiStick\n1.0" (at 124.968 106.68) (layer F.SilkS)
+  (gr_text "espStick\n1.0" (at 124.968 106.68) (layer F.SilkS)
     (effects (font (size 1.27 1.143) (thickness 0.1524)))
   )

Commit message: RESET label added
Other:
- board text added: "RESET"
Changed lines of the file:
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@@
-(kicad_pcb (version 4) (host pcbnew 0.201512201246+6385~39~ubuntu14.04.1-stable)
+(kicad_pcb (version 4) (host pcbnew 0.201511131146+6311~30~ubuntu14.04.1-product)
   (general
     (links 58)
@@
     (area 108.553467 47.946859 141.512074 116.7956)
     (thickness 1.6002)
-    (drawings 42)
+    (drawings 43)
     (tracks 529)
     (zones 0)
@@
     (descr "Through hole pin header")
     (tags "pin header")
-    (fp_text reference P2 (at 2.2098 8.9662 90) (layer F.SilkS)
+    (fp_text reference P2 (at 0.7366 3.5306 90) (layer F.SilkS) hide
       (effects (font (size 1 1) (thickness 0.15)))
     )
@@
       (net 9 /ESP_TXD))
   )
+  (gr_text RESET (at 118.2116 95.7834) (layer F.SilkS)
+    (effects (font (size 1.27 1.016) (thickness 0.1524)))
+  )
   (gr_text +5V (at 117.856 105.41) (layer F.SilkS)

Commit message: Attaching GPIO15 to panStamp's RESET line
Connections:
- P1 pad 4: /PS_RESET -> /GPIO15
- PS1 pad 12: /PS_RESET -> /GPIO15
Routing:
- net /GPIO15: track 22.4 -> 51.3 mm, vias 2 -> 6
- net /PS_RESET: track 27.6 -> 0.00 mm, vias 3 -> 0

Commit message: Version 1.0 released
Parts:
- removed ANT1: ANTENNA, myconnectors:SMA_RightAngle_Tyco
- removed the G*** at (121.9, 83.3)
- removed P2: CONN_01X07, Pin_Headers:Pin_Header_Straight_1x07
- removed the fiducial at (115.8, 109.5)
- removed the fiducial at (134.9, 57.1)
- added D3: D_Schottky_x2_ACom_KKA, mysmd:SOT23, F.Cu at (89.8, 82.2)
- added D4: BAS16, SOD323, F.Cu at (89.9, 85.9)
- added G***: PANSTAMPLOGO, mymods:PANSTAMPLOGO, F.Cu at (62.3, 117.1)
- added G***: PANSTAMPLOGO, mymods:PANSTAMPLOGO, F.Cu at (85.6, 127.5)
- added G***: LOGO, mysmd:oshlogo, F.Cu at (97.1, 100.7)
- added PS2: PANSTAMP_MINIBAT, mymods:minibat, F.Cu at (76.0, 120.1)
- added U4: LY-SK10, LY-SK10, F.Cu at (85.3, 100.9)
- added fiducial: VAL**, mymods:fiducial, F.Cu at (54.2, 137.1)
- added fiducial: VAL**, mymods:fiducial, F.Cu at (100.8, 76.0)
- P1: value CONN_01X07 -> CONN_01X02; footprint Pin_Headers:Pin_Header_Straight_1x07 -> Pin_Headers:Pin_Header_Straight_1x02
- P3: footprint Pin_Headers:Pin_Header_Straight_1x02 -> myconnectors:PWR_3A
- U2: footprint mysmd:ESP-12E -> ESP-12E; moved to F.Cu
- U3: value LY-SK10 -> ANTENNA; footprint mysmd:LY-SK10 -> myconnectors:SMA_RightAngle_Tyco
- moved U3 80.3 mm to (52.9, 120.1), turned to 90 degrees
- moved PS1 70.2 mm to (70.1, 120.0), turned to 90 degrees
- moved R2 68.6 mm to (57.6, 101.9), turned to 270 degrees
- moved U2 60.6 mm to (56.6, 97.6), turned to 90 degrees
- moved SW1 58.2 mm to (73.6, 102.9)
- moved SW2 57.6 mm to (62.6, 102.9)
- moved D2 52.2 mm to (75.0, 82.1), turned to 270 degrees
- moved R3 50.6 mm to (75.0, 86.0), turned to 90 degrees
- moved R5 50.3 mm to (76.6, 82.1), turned to 270 degrees
- moved R1 49.3 mm to (76.6, 86.0), turned to 90 degrees
- moved C4 46.3 mm to (79.0, 86.0)
- moved P1 46.3 mm to (90.2, 90.9), turned to 270 degrees
- moved D1 46.2 mm to (78.2, 82.1), turned to 270 degrees
- moved R4 45.2 mm to (79.8, 82.1), turned to 270 degrees
- moved C3 43.4 mm to (80.6, 86.0)
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Connections:
- P1 pad 1: /PS_RXD -> +5V
- P1 pad 2: /PS_TXD -> GND
- P3 pad 1: Net-(C1-Pad1) -> +5V
- PS1 pad 31: /TOANT -> Net-(PS1-Pad31)
- SW1 pad 1: GND -> /GPIO0
- SW1 pad 2: /GPIO0 -> GND
- U3 pad 1: /PS_TXD -> Net-(PS1-Pad31)
- U3 pad 2: /ESP_RXD -> GND
Routing:
- net GND: track 223.9 -> 720.1 mm, vias 82 -> 216
- net VCC: track 78.9 -> 114.0 mm, vias 3 -> 0
- net /GPIO15: track 51.3 -> 78.2 mm
- net /ESP_RESET: track 29.3 -> 7.83 mm, vias 5 -> 0
- net +5V: track 0.00 -> 19.3 mm
- net Net-(R1-Pad1): track 12.7 -> 25.5 mm, vias 1 -> 4
- net Net-(D1-Pad2): track 13.0 -> 21.7 mm, vias 1 -> 0
- net Net-(D2-Pad2): track 8.47 -> 15.2 mm, vias 1 -> 0
- net Net-(PS1-Pad31): track 0.00 -> 6.14 mm
- net /PS_RXD: track 22.1 -> 16.0 mm, vias 1 -> 0
- net /ESP_RXD: track 39.4 -> 45.3 mm, vias 1 -> 2
- net /TOANT: track 5.87 -> 0.00 mm
- net /ESP_TXD: track 39.4 -> 42.2 mm, vias 1 -> 2
- net Net-(C1-Pad1): track 8.03 -> 5.29 mm
- net /GPIO0: track 22.9 -> 24.6 mm
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Other:
- board size 25.4 x 55.8 mm -> 58.1 x 64.2 mm
- board text added: "ESP-12E wifi module"
- board text added: "GPIO0"
- board text added: "LIBERIOT WiFi gateway 1.0"
- board text added: "Long-range radio (NRG)"
- board text added: "NRG"
- board text added: "www.liberiot.org"
- board text removed: "3.3V"
- board text removed: "espStick 1.0"
- board text removed: "www.panstamp.com"

Commit message: New 1.1 version fixing 1.0
Parts:
- added PROG1: CONN_01X07, Pin_Headers:Pin_Header_Straight_1x07, F.Cu at (59.0, 78.5)
- C2: value 10u -> 1u
- U1: value MCP1702 -> AP7365; footprint libcms:SOT23 -> TO_SOT_Packages_SMD:SOT-23-5
- moved C2 4.21 mm to (86.4, 86.0), turned to 90 degrees
- moved U1 1.60 mm to (83.3, 86.0)
- moved C1 0.31 mm to (87.9, 86.0)
- turned C3 to 90 degrees
- turned C4 to 90 degrees
Connections:
- C2 pad 1: VCC -> Net-(C1-Pad1)
- PS1 pad 12: /GPIO15 -> /GPIO14
- PS2 pad 18: /GPIO15 -> /GPIO14
- U1 pad 1: GND -> Net-(C1-Pad1)
- U1 pad 2: VCC -> GND
- U2 pad 5: Net-(U2-Pad5) -> /GPIO14
Routing:
- net /GPIO14: track 0.00 -> 68.0 mm, vias 0 -> 6
- net /GPIO15: track 78.2 -> 17.8 mm, vias 6 -> 2
- net /ESP_RESET: track 7.83 -> 36.0 mm, vias 0 -> 1
- net GND: track 720.1 -> 702.8 mm, vias 216 -> 212
- net VCC: track 114.0 -> 130.4 mm
- net /GPIO0: track 24.6 -> 37.1 mm
- net /ESP_TXD: track 42.2 -> 52.4 mm
- net Net-(C1-Pad1): track 5.29 -> 9.10 mm
- net /ESP_RXD: track 45.3 -> 48.7 mm
Other:
- board text added: "0"
- board text added: "15"
- board text added: "LIBERIOT WiFi gateway 1.1"
- board text added: "RST"
- board text added: "RXD"
- board text added: "TXD"
- board text added: "VCC"
- board text removed: "LIBERIOT WiFi gateway 1.0"
