File: esp-touch/esp-touch.kicad_pcb (KiCad board)
At the start: 2 copper layers, 113 x 180 mm, 64 parts, among them P1 CONN_01X02, P2 CONN_01X05, P3 DISPLAY, P4 CONN_01X03, P5 CONN_01X02, P6 CONN_01X02, P7 CONN_01X04, Q1 Q_NMOS_GSD, SW1 SW_PUSH_SMALL, SW2 SW_PUSH_SMALL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

Commit message: Multiple mistakes fixed
Parts:
- removed P5: CONN_01X02, Pin_Headers:Pin_Header_Straight_1x02
- added G***: PANSTAMPLOGO, mymods:PANSTAMPLOGO, B.Cu at (237.0, 86.5)
- added G***: LOGO, mymods:oshlogo, B.Cu at (229.9, 106.3)
- added Q2: Q_NPN_EBC, mysmd:SOT23EBC, F.Cu at (256.0, 91.8)
- added R18: 2k2, mysmd:SM0603S, F.Cu at (251.9, 91.0)
- added SP1: AL11P, mymods:Buzzer_7.6_12.0, F.Cu at (265.2, 92.4)
- P2: footprint mysmd:microUSB_female -> mysmd:MICRO_USB_SOCKET
- moved G*** 51.9 mm to (230.0, 131.7)
- moved G*** 34.0 mm to (222.6, 113.7)
- moved R16 9.20 mm to (269.7, 85.0), turned to 180 degrees
Connections:
- R16 pad 1: Net-(P5-Pad1) -> VCC
- R16 pad 2: /GPIO15 -> Net-(R16-Pad2)
Routing:
- net /GPIO15: track 86.1 -> 50.5 mm
- net +5V: track 71.6 -> 57.6 mm
- net GND: track 363.7 -> 372.8 mm, vias 124 -> 125
- net Net-(R16-Pad2): track 0.00 -> 7.42 mm
- net Net-(Q2-Pad3): track 0.00 -> 4.62 mm
- net Net-(P5-Pad1): track 2.93 -> 0.00 mm
- net (no net): track 0.00 -> 2.93 mm
- net Net-(Q2-Pad2): track 0.00 -> 2.39 mm
- net Net-(C7-Pad1): track 12.1 -> 12.8 mm
- net VCC: track 216.9 -> 217.6 mm
- net Net-(C8-Pad1): track 11.2 -> 11.0 mm, vias 0 -> 2
Other:
- rule pad_to_mask_clearance: 0.0762 -> 0
- board text added: "RXD"
- board text added: "TXD"
- board text added: "V.0.2"
- board text removed: "GND BZ"
- board text removed: "V.0.1"
