File: panstamp-nrg3/psu.sch (KiCad schematic (older format))
At the start: 22 parts, among them J1 MicroUSB, J2 PWR, Q1 DMG3415U, Q3 DMG3415U, U3 MCP1640B, U4 AP7365-3.0

Commit message: Cahnging MBR120 by RB168MM-40TR
Parts:
- D6: value MBR120 -> RB168MM-40TR
- U4: value AP7365-3.0 -> AP7365-3.3
Changed lines of the file:
@@
 P 7850 2400
 F 0 "U4" H 7950 2150 60  0000 C CNN
-F 1 "AP7365-3.0" H 7850 2650 60  0000 C CNN
+F 1 "AP7365-3.3" H 7850 2650 60  0000 C CNN
 F 2 "TO_SOT_Packages_SMD:SOT-23-5" H 7850 2350 60  0001 C CNN
 F 3 "" H 7850 2350 60  0000 C CNN
@@
 P 4000 4450
 F 0 "D6" H 4000 4350 50  0000 C CNN
-F 1 "MBR120" H 4000 4550 50  0000 C CNN
+F 1 "RB168MM-40TR" H 4000 4550 50  0000 C CNN
 F 2 "smd-semi:SOD-123" H 4000 4450 50  0001 C CNN
 F 3 "" H 4000 4450 50  0001 C CNN
