File: panstamp-nrg3/panstamp.sch (KiCad schematic (older format))
At the start: 67 parts, among them SW1 RESET, U1 CC430F5137, U14 B3725, U15 CC1190, X1 26MHz, X2 32.768KHz

Commit message: New comments
Other:
- note added: "SAW filter bypass\n(assembled by default)"
- note removed: "SAW filter bypass"
Changed lines of the file:
@@
 $EndComp
 Text Notes 9000 2425 2    39   ~ 0
-SAW filter bypass
+SAW filter bypass\n(assembled by default)
 Connection ~ 6750 1525
 Wire Wire Line
